File: Module/AttendanceBot2000/AB2KController.sch (EAGLE design)
At the start: 3 parts

Commit message: Schematic and layout WIP.
Parts:
- removed FRAME1: FRAME-LEDGER, SparkFun-Aesthetics:FRAME-LEDGER
- added C1, C11, C2, C3, C4, C5: 0.15, resistor:C-USC1206K
- added C10: 10uF, rcl:CPOL-USD/7343-31R
- added C6, C7: 10, resistor:CPOL-USD/7343-31W
- added C8: 220uF, rcl:CPOL-USD/7343-31R
- added C9: 0.056uF, rcl:C-USC1210
- added D1: PMEG3030EP, kb1vc_robot_parts:PMEG3030EP
- added IC1, IC2: 74AHCT1G04DBV, 74xx-little-de:74AHCT1G04DBV
- added IC3: LM386M-1, linear:LM386M-1
- added JP1: WAVtrg Right, SparkFun-Connectors:M11PTH
- added JP10: TRAIN_ENA, pinhead:PINHD-1X2
- added JP2: WAVtrg Left, SparkFun-Connectors:M11PTH
- added JP3, JP5: L_MOT, SparkFun-Connectors:M025MM
- added JP4: BAT, SparkFun-Connectors:M025MM
- added JP6: R_MOT, SparkFun-Connectors:M025MM
- added JP7: GND_SEL_SERIAL, pinhead:PINHD-1X2
- added JP8: GO_BUTTON_IN, SparkFun-Connectors:M025MM
- added JP9: FTDI Basic Prog. Port, SparkFun-Connectors:ARDUINO_SERIAL_PROGRAMPTH
- added R1, R3, R5, R7, R9: 100, resistor:R-US_M1206
- added R10, R2, R4, R6, R8: 10K, resistor:R-US_M1206
- added R21: 10, rcl:R-US_R1210
- added R22, R23: 5K, rcl:R-US_R1206
- added U$2, U$3, U$4, U$5, U$6: TCRT5000, kb1vc_robot_parts:TCRT5000
- added U1: L298, SparkFun-PowerIC:L298
- added U2, U3, U4, U5, U6: QRE1113, SparkFun-Sensors:QRE1113
Connections:
- new net AUDIO_RESET: JP2.11, U$1.4
- new net AUD_RXD: JP1.6, U$1.*6
- new net AUD_TXD: JP1.7, U$1.*5
- new net DIRA_H: IC1A.I, U$1.12, U1.IN1
- new net DIRA_L: IC1A.O, U1.IN2
- new net DIRB_H: IC2A.I, U$1.13, U1.IN3
- new net DIRB_L: IC2A.O, U1.IN4
- new net DTR: JP9.DTR, U$1.DTR
- new net GND: C1.2, C11.2, C2.2, C3.2, C4.2, C5.2, C6.-, C7.-, IC3.-IN, IC3.GND, JP1.1, JP1.10, JP1.4, JP10.2, JP2.1, JP3.2, JP4.2, JP7.2, JP8.2, JP9.CTS, JP9.GND, R21.1, R23.1, U$1.GND, U$1.GND@2, U$2.CAT, U$2.E, U$3.CAT, U$3.E, U$4.CAT, U$4.E, U$5.CAT, U$5.E, U$6.CAT, U$6.E, U1.CSA, U1.CSB, U1.GND, U2.E, U2.K, U3.E, U3.K, U4.E, U4.K, U5.E, U5.K, U6.E, U6.K
- new net L_PWM: U$1.*3, U1.ENA
- new net N$1: JP5.1, U1.OUT1
- new net N$11: R5.1, U$4.ANO, U4.A
- new net N$13: R7.1, U$3.ANO, U3.A
- new net N$14: R9.1, U$2.ANO, U2.A
- new net N$16: IC3.+IN, R22.2, R23.2
- new net N$18: C8.+, C9.1, IC3.OUT
- new net N$19: C8.-, JP3.1
- new net N$2: JP5.2, U1.OUT2
- new net N$20: C10.-, IC3.GAIN@2
- new net N$21: C9.2, R21.2
- new net N$22: C10.+, IC3.GAIN@1
- new net N$23: C11.1, IC3.BYPASS
- new net N$25: JP8.1, U$1.2
- new net N$27: JP1.3, R22.1
- new net N$28: JP1.5, JP7.1
- new net N$3: JP6.1, U1.OUT3
- new net N$4: JP6.2, U1.OUT4
- new net N$5: D1.A, JP4.1
- new net N$7: R1.1, U$6.ANO, U6.A
- new net N$8: R3.1, U$5.ANO, U5.A
- new net RXD_TTL: JP9.TXO, U$1.RXI
- new net R_PWM: U$1.*11, U1.ENB
- new net SEN_0: R2.1, U$1.A0, U$6.C, U6.C
- new net SEN_1: R4.1, U$1.A1, U$5.C, U5.C
- new net SEN_2: R6.1, U$1.A2, U$4.C, U4.C
- new net SEN_3: R8.1, U$1.A3, U$3.C, U3.C
- new net SEN_4: R10.1, U$1.A4, U$2.C, U2.C
- new net TRAIN_L: JP10.1, U$1.7
- new net TXD_TTL: JP9.RXI, U$1.TXO
- new net VCC: C1.1, C2.1, C3.1, C4.1, C5.1, C6.+, C7.+, JP1.11, JP9.VCC, R1.2, R10.2, R2.2, R3.2, R4.2, R5.2, R6.2, R7.2, R8.2, R9.2, U$1.VCC, U1.VLS
- new net V_IN: D1.C, IC3.VS, U$1.RAW, U1.VS
Other:
- note added: "0.15uF caps from local reel"
- note added: "10uF caps from local reel"
- note added: "A"
- note added: "Matt Reilly"
- note added: "Option 1 -- Short Range Sensors"
- note added: "Option 2 -- Long Range Sensors"
- note added: "separate by 800 mils"
- moved on the sheet: U$1

Commit message: More progress on routing
Parts:
- added JP11: GO_LIGHT, SparkFun-Connectors:M025MM
- added Q1, Q2, Q3, Q4, Q5, Q6: 2N3904, transistor-npn:2N3904
- added R11, R12, R13, R14, R15, R16: 1K, resistor:R-US_M1206
Connections:
- new net GO_IN: JP8.1, U$1.*10
- new net GO_LT_ON: R16.2, U$1.*9
- new net N$10: Q2.E, R3.2
- new net N$12: Q3.E, R5.2
- new net N$15: Q1.B, R11.1
- new net N$17: Q2.B, R12.1
- new net N$24: Q3.B, R13.1
- new net N$26: Q4.B, R14.1
- new net N$29: Q5.B, R15.1
- new net N$30: Q4.E, R7.2
- new net N$31: Q5.E, R9.2
- new net N$6: JP11.1, Q6.C
- new net N$9: Q1.E, R1.2
- net GND: now also Q6.E
- net N$25: now also Q6.B, R16.1; no longer JP8.1, U$1.2
- net SEN_0: now also U$1.A1; no longer U$1.A0
- net SEN_1: now also U$1.A0; no longer U$1.A1
- net VCC: now also R11.2, R12.2, R13.2, R14.2, R15.2; no longer R1.2, R3.2, R5.2, R7.2, R9.2
- net V_IN: now also JP11.2, Q1.C, Q2.C, Q3.C, Q4.C, Q5.C
Other:
- note added: "Note swap of Sen 0 and Sen 1 for routing convenience"
- moved on the sheet: C1, C2, C3, C4, C5, C6, C7, R1, R10, R2, R3, R4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

Commit message: More layout complete
Parts:
- removed C4, C5: 0.15, resistor:C-USC1206K
- removed C6, C7: 10, resistor:CPOL-USD/7343-31W
- removed JP9: FTDI Basic Prog. Port, SparkFun-Connectors:ARDUINO_SERIAL_PROGRAMPTH
Connections:
- removed net DTR: JP9.DTR, U$1.DTR
- net GND: no longer C4.2, C5.2, C6.-, C7.-, JP9.CTS, JP9.GND
- net RXD_TTL: no longer JP9.TXO
- net SEN_3: now also U$1.A6; no longer U$1.A3
- net SEN_4: now also U$1.A7; no longer U$1.A4
- net TXD_TTL: no longer JP9.RXI
- net VCC: no longer C4.1, C5.1, C6.+, C7.+, JP9.VCC
Other:
- note removed: "10uF caps from local reel"
- moved on the sheet: Q6, R16
Changed lines of the file:
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@@
 <part name="C2" library="resistor" deviceset="C-US" device="C1206K" value="0.15"/>
 <part name="C3" library="resistor" deviceset="C-US" device="C1206K" value="0.15"/>
-<part name="C4" library="resistor" deviceset="C-US" device="C1206K" value="0.15"/>
-<part name="C5" library="resistor" deviceset="C-US" device="C1206K" value="0.15"/>
-<part name="C6" library="resistor" deviceset="CPOL-US" device="D/7343-31W" value="10"/>
-<part name="C7" library="resistor" deviceset="CPOL-US" device="D/7343-31W" value="10"/>
 <part name="SUPPLY11" library="supply2" deviceset="GND" device=""/>
 <part name="SUPPLY12" library="SparkFun-Aesthetics" deviceset="VCC" device=""/>
-<part name="JP9" library="SparkFun-Connectors" deviceset="ARDUINO_SERIAL_PROGRAM" device="PTH" value="FTDI Basic Prog. Port"/>
-<part name="SUPPLY13" library="SparkFun-Aesthetics" deviceset="VCC" device=""/>
-<part name="GND8" library="supply1" deviceset="GND" device=""/>
 <part name="JP1" library="SparkFun-Connectors" deviceset="M11" device="PTH" value="WAVtrg Right"/>
 <part name="JP2" library="SparkFun-Connectors" deviceset="M11" device="PTH" value="WAVtrg Left"/>
@@
 <text x="-210.82" y="60.96" size="1.778" layer="91">Option 1 -- Short Range Sensors</text>
 <text x="-210.82" y="33.02" size="1.778" layer="91">Option 2 -- Long Range Sensors</text>
-<text x="-45.72" y="78.74" size="1.778" layer="91">10uF caps from local reel</text>
 <text x="-45.72" y="73.66" size="1.778" layer="91">0.15uF caps from local reel</text>
 <text x="-149.86" y="210.82" size="1.778" layer="91">separate by 800 mils</text>
@@
 <instance part="C2" gate="G$1" x="-66.04" y="88.9"/>
 <instance part="C3" gate="G$1" x="-55.88" y="88.9"/>
-<instance part="C4" gate="G$1" x="-45.72" y="88.9"/>
-<instance part="C5" gate="G$1" x="-35.56" y="88.9"/>
-<instance part="C6" gate="G$1" x="-25.4" y="88.9"/>
-<instance part="C7" gate="G$1" x="-12.7" y="88.9"/>
 <instance part="SUPPLY11" gate="GND" x="-76.2" y="78.74"/>
 <instance part="SUPPLY12" gate="G$1" x="-76.2" y="96.52"/>
-<instance part="JP9" gate="G$1" x="-236.22" y="132.08"/>
-<instance part="SUPPLY13" gate="G$1" x="-220.98" y="139.7"/>
-<instance part="GND8" gate="1" x="-226.06" y="137.16"/>
 <instance part="JP1" gate="G$1" x="-134.62" y="190.5"/>
 <instance part="JP2" gate="G$1" x="-144.78" y="190.5" rot="MR0"/>
@@
 <instance part="R14" gate="G$1" x="-175.26" y="109.22" rot="R90"/>
 <instance part="R15" gate="G$1" x="-152.4" y="109.22" rot="R90"/>
-<instance part="Q6" gate="G1" x="-121.92" y="129.54" smashed="yes">
-<attribute name="NAME" x="-119.38" y="129.54" size="1.778" layer="95"/>
-<attribute name="VALUE" x="-116.84" y="124.46" size="1.778" layer="96"/>
+<instance part="Q6" gate="G1" x="-119.38" y="129.54" smashed="yes">
+<attribute name="NAME" x="-116.84" y="129.54" size="1.778" layer="95"/>
+<attribute name="VALUE" x="-114.3" y="124.46" size="1.778" layer="96"/>
 </instance>
 <instance part="JP11" gate="G$1" x="-106.68" y="137.16" rot="MR0"/>
-<instance part="SUPPLY10" gate="GND" x="-119.38" y="119.38"/>
-<instance part="R16" gate="G$1" x="-132.08" y="129.54" rot="R180"/>
+<instance part="SUPPLY10" gate="GND" x="-116.84" y="119.38"/>
+<instance part="R16" gate="G$1" x="-129.54" y="129.54" rot="R180"/>
 </instances>
 <busses>
@@
 </segment>
 <segment>
-<pinref part="C7" gate="G$1" pin="-"/>
-<pinref part="C6" gate="G$1" pin="-"/>
-<wire x1="-12.7" y1="83.82" x2="-25.4" y2="83.82" width="0.1524" layer="91"/>
-<pinref part="C5" gate="G$1" pin="2"/>
-<wire x1="-25.4" y1="83.82" x2="-35.56" y2="83.82" width="0.1524" layer="91"/>
-<pinref part="C4" gate="G$1" pin="2"/>
-<wire x1="-35.56" y1="83.82" x2="-45.72" y2="83.82" width="0.1524" layer="91"/>
 <pinref part="C3" gate="G$1" pin="2"/>
-<wire x1="-45.72" y1="83.82" x2="-55.88" y2="83.82" width="0.1524" layer="91"/>
 <pinref part="C2" gate="G$1" pin="2"/>
 <wire x1="-55.88" y1="83.82" x2="-66.04" y2="83.82" width="0.1524" layer="91"/>
@@
 <pinref part="SUPPLY11" gate="GND" pin="GND"/>
 <wire x1="-76.2" y1="83.82" x2="-76.2" y2="81.28" width="0.1524" layer="91"/>
-<junction x="-25.4" y="83.82"/>
-<junction x="-35.56" y="83.82"/>
-<junction x="-55.88" y="83.82"/>
-<junction x="-45.72" y="83.82"/>
 <junction x="-66.04" y="83.82"/>
 <junction x="-76.2" y="83.82"/>
-</segment>
-<segment>
-<pinref part="JP9" gate="G$1" pin="GND"/>
-<wire x1="-231.14" y1="139.7" x2="-228.6" y2="139.7" width="0.1524" layer="91"/>
-<pinref part="JP9" gate="G$1" pin="CTS"/>
-<wire x1="-228.6" y1="139.7" x2="-226.06" y2="139.7" width="0.1524" layer="91"/>
-<wire x1="-231.14" y1="137.16" x2="-228.6" y2="137.16" width="0.1524" layer="91"/>
-<wire x1="-228.6" y1="137.16" x2="-228.6" y2="139.7" width="0.1524" layer="91"/>
-<pinref part="GND8" gate="1" pin="GND"/>
-<junction x="-228.6" y="139.7"/>
 </segment>
 <segment>
@@
 <pinref part="Q6" gate="G1" pin="E"/>
 <pinref part="SUPPLY10" gate="GND" pin="GND"/>
-<wire x1="-119.38" y1="124.46" x2="-119.38" y2="121.92" width="0.1524" layer="91"/>
+<wire x1="-116.84" y1="124.46" x2="-116.84" y2="121.92" width="0.1524" layer="91"/>
 </segment>
 </net>
@@
 <pinref part="C3" gate="G$1" pin="1"/>
 <wire x1="-66.04" y1="91.44" x2="-55.88" y2="91.44" width="0.1524" layer="91"/>
-<pinref part="C4" gate="G$1" pin="1"/>
-<wire x1="-55.88" y1="91.44" x2="-45.72" y2="91.44" width="0.1524" layer="91"/>
-<pinref part="C5" gate="G$1" pin="1"/>
-<wire x1="-45.72" y1="91.44" x2="-35.56" y2="91.44" width="0.1524" layer="91"/>
-<pinref part="C6" gate="G$1" pin="+"/>
-<wire x1="-35.56" y1="91.44" x2="-25.4" y2="91.44" width="0.1524" layer="91"/>
-<pinref part="C7" gate="G$1" pin="+"/>
-<wire x1="-25.4" y1="91.44" x2="-12.7" y2="91.44" width="0.1524" layer="91"/>
 <junction x="-76.2" y="91.44"/>
 <junction x="-66.04" y="91.44"/>
-<junction x="-55.88" y="91.44"/>
-<junction x="-45.72" y="91.44"/>
-<junction x="-35.56" y="91.44"/>
-<junction x="-25.4" y="91.44"/>
-</segment>
-<segment>
-<pinref part="JP9" gate="G$1" pin="VCC"/>
-<wire x1="-231.14" y1="134.62" x2="-220.98" y2="134.62" width="0.1524" layer="91"/>
-<wire x1="-220.98" y1="134.62" x2="-220.98" y2="139.7" width="0.1524" layer="91"/>
-<pinref part="SUPPLY13" gate="G$1" pin="VCC"/>
 </segment>
 <segment>
@@
 </segment>
 <segment>
-<pinref part="U$1" gate="G$1" pin="A3"/>
-<wire x1="-165.1" y1="154.94" x2="-157.48" y2="154.94" width="0.1524" layer="91"/>
-<label x="-157.48" y="154.94" size="1.27" layer="95" xref="yes"/>
+<label x="-157.48" y="129.54" size="1.27" layer="95" xref="yes"/>
+<pinref part="U$1" gate="G$1" pin="A6"/>
+<wire x1="-165.1" y1="129.54" x2="-157.48" y2="129.54" width="0.1524" layer="91"/>
 </segment>
 <segment>
@@
 </segment>
 <segment>
-<pinref part="U$1" gate="G$1" pin="A4"/>
-<wire x1="-187.96" y1="132.08" x2="-190.5" y2="132.08" width="0.1524" layer="91"/>
-<label x="-190.5" y="132.08" size="1.27" layer="95" rot="R180" xref="yes"/>
+<label x="-157.48" y="132.08" size="1.27" layer="95" xref="yes"/>
+<pinref part="U$1" gate="G$1" pin="A7"/>
+<wire x1="-157.48" y1="132.08" x2="-165.1" y2="132.08" width="0.1524" layer="91"/>
 </segment>
 <segment>
@@
 <net name="TXD_TTL" class="0">
 <segment>
-<pinref part="JP9" gate="G$1" pin="RXI"/>
-<wire x1="-231.14" y1="129.54" x2="-226.06" y2="129.54" width="0.1524" layer="91"/>
-<label x="-226.06" y="129.54" size="1.27" layer="95" xref="yes"/>
-</segment>
-<segment>
 <pinref part="U$1" gate="G$1" pin="TXO"/>
 <wire x1="-187.96" y1="165.1" x2="-190.5" y2="165.1" width="0.1524" layer="91"/>
@@
 <net name="RXD_TTL" class="0">
 <segment>
-<pinref part="JP9" gate="G$1" pin="TXO"/>
-<wire x1="-231.14" y1="132.08" x2="-226.06" y2="132.08" width="0.1524" layer="91"/>
-<label x="-226.06" y="132.08" size="1.27" layer="95" xref="yes"/>
-</segment>
-<segment>
 <pinref part="U$1" gate="G$1" pin="RXI"/>
 <wire x1="-187.96" y1="162.56" x2="-190.5" y2="162.56" width="0.1524" layer="91"/>
 <label x="-190.5" y="162.56" size="1.27" layer="95" rot="R180" xref="yes"/>
-</segment>
-</net>
-<net name="DTR" class="0">
-<segment>
-<pinref part="JP9" gate="G$1" pin="DTR"/>
-<wire x1="-231.14" y1="127" x2="-226.06" y2="127" width="0.1524" layer="91"/>
-<label x="-226.06" y="127" size="1.27" layer="95" xref="yes"/>
-</segment>
-<segment>
-<pinref part="U$1" gate="G$1" pin="DTR"/>
-<wire x1="-187.96" y1="170.18" x2="-190.5" y2="170.18" width="0.1524" layer="91"/>
-<label x="-190.5" y="170.18" size="1.27" layer="95" rot="R180" xref="yes"/>
 </segment>
 </net>
@@
 <segment>
 <pinref part="JP11" gate="G$1" pin="1"/>
-<wire x1="-114.3" y1="137.16" x2="-119.38" y2="137.16" width="0.1524" layer="91"/>
+<wire x1="-114.3" y1="137.16" x2="-116.84" y2="137.16" width="0.1524" layer="91"/>
 <pinref part="Q6" gate="G1" pin="C"/>
-<wire x1="-119.38" y1="137.16" x2="-119.38" y2="134.62" width="0.1524" layer="91"/>
+<wire x1="-116.84" y1="137.16" x2="-116.84" y2="134.62" width="0.1524" layer="91"/>
 </segment>
 </net>
@@
 <pinref part="Q6" gate="G1" pin="B"/>
 <pinref part="R16" gate="G$1" pin="1"/>
-<wire x1="-124.46" y1="129.54" x2="-127" y2="129.54" width="0.1524" layer="91"/>
+<wire x1="-121.92" y1="129.54" x2="-124.46" y2="129.54" width="0.1524" layer="91"/>
 </segment>
 </net>
@@
 <segment>
 <pinref part="R16" gate="G$1" pin="2"/>
-<wire x1="-137.16" y1="129.54" x2="-139.7" y2="129.54" width="0.1524" layer="91"/>
-<label x="-139.7" y="129.54" size="1.27" layer="95" rot="R180" xref="yes"/>
-</segment>
-<segment>
+<wire x1="-134.62" y1="129.54" x2="-137.16" y2="129.54" width="0.1524" layer="91"/>
+<label x="-137.16" y="129.54" size="1.27" layer="95" rot="R180" xref="yes"/>
+</segment>
+<segment>

Commit message: Finished routing.  Sleep on it for a day
Parts:
- removed FRAME2: FRAME-LETTER, SparkFun-Aesthetics:FRAME-LETTER
- added JP9: SERIAL, SparkFun-Connectors:M03PTH
- JP3: value L_MOT -> SPKR
Connections:
- net GND: now also JP9.2
- net RXD_TTL: now also JP9.1
- net TXD_TTL: now also JP9.3
Changed lines of the file:
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@@
 <?xml version="1.0" encoding="utf-8"?>
 <!DOCTYPE eagle SYSTEM "eagle.dtd">
-<eagle version="7.3.0">
+<eagle version="7.5.0">
 <drawing>
 <settings>
@@
 <setting verticaltext="up"/>
 </settings>
-<grid distance="0.1" unitdist="inch" unit="inch" style="lines" multiple="1" display="yes" altdistance="0.01" altunitdist="inch" altunit="inch"/>
+<grid distance="0.1" unitdist="inch" unit="inch" style="lines" multiple="1" display="no" altdistance="0.01" altunitdist="inch" altunit="inch"/>
 <layers>
 <layer number="1" name="Top" color="4" fill="1" visible="no" active="no"/>
+<layer number="2" name="Route2" color="1" fill="3" visible="no" active="no"/>
+<layer number="3" name="Route3" color="4" fill="3" visible="no" active="no"/>
+<layer number="14" name="Route14" color="1" fill="6" visible="no" active="no"/>
+<layer number="15" name="Route15" color="4" fill="6" visible="no" active="no"/>
 <layer number="16" name="Bottom" color="1" fill="1" visible="no" active="no"/>
 <layer number="17" name="Pads" color="2" fill="1" visible="no" active="no"/>
@@
 </classes>
 <parts>
-<part name="FRAME2" library="SparkFun-Aesthetics" deviceset="FRAME-LETTER" device=""/>
 <part name="U$1" library="kb1vc_Arduino_Parts" deviceset="ARDUINO_PRO_MINI" device=""/>
 <part name="JP4" library="SparkFun-Connectors" deviceset="M02" device="5MM" value="BAT"/>
@@
 <part name="JP2" library="SparkFun-Connectors" deviceset="M11" device="PTH" value="WAVtrg Left"/>
 <part name="IC3" library="linear" deviceset="LM386?-*" device="M" technology="1"/>
-<part name="JP3" library="SparkFun-Connectors" deviceset="M02" device="5MM" value="L_MOT"/>
+<part name="JP3" library="SparkFun-Connectors" deviceset="M02" device="5MM" value="SPKR"/>
 <part name="SUPPLY14" library="supply2" deviceset="GND" device=""/>
 <part name="SUPPLY15" library="supply2" deviceset="GND" device=""/>
@@
 <part name="SUPPLY10" library="supply2" deviceset="GND" device=""/>
 <part name="R16" library="resistor" deviceset="R-US_" device="M1206" value="1K"/>
+<part name="JP9" library="SparkFun-Connectors" deviceset="M03" device="PTH" value="SERIAL"/>
+<part name="SUPPLY13" library="supply2" deviceset="GND" device=""/>
 </parts>
 <sheets>
@@
 </plain>
 <instances>
-<instance part="FRAME2" gate="G$1" x="-251.46" y="30.48"/>
-<instance part="FRAME2" gate="V" x="-104.14" y="30.48"/>
 <instance part="U$1" gate="G$1" x="-177.8" y="149.86"/>
 <instance part="JP4" gate="G$1" x="-233.68" y="198.12" rot="MR180"/>
@@
 <instance part="SUPPLY10" gate="GND" x="-116.84" y="119.38"/>
 <instance part="R16" gate="G$1" x="-129.54" y="129.54" rot="R180"/>
+<instance part="JP9" gate="G$1" x="-203.2" y="182.88"/>
+<instance part="SUPPLY13" gate="GND" x="-193.04" y="175.26"/>
 </instances>
 <busses>
@@
 <pinref part="SUPPLY10" gate="GND" pin="GND"/>
 <wire x1="-116.84" y1="124.46" x2="-116.84" y2="121.92" width="0.1524" layer="91"/>
+</segment>
+<segment>
+<pinref part="JP9" gate="G$1" pin="2"/>
+<wire x1="-195.58" y1="182.88" x2="-193.04" y2="182.88" width="0.1524" layer="91"/>
+<pinref part="SUPPLY13" gate="GND" pin="GND"/>
+<wire x1="-193.04" y1="182.88" x2="-193.04" y2="177.8" width="0.1524" layer="91"/>
 </segment>
 </net>
@@
 <label x="-190.5" y="165.1" size="1.27" layer="95" rot="R180" xref="yes"/>
 </segment>
+<segment>
+<pinref part="JP9" gate="G$1" pin="3"/>
+<wire x1="-195.58" y1="185.42" x2="-190.5" y2="185.42" width="0.1524" layer="91"/>
+<label x="-190.5" y="185.42" size="1.27" layer="95" xref="yes"/>
+</segment>
 </net>
 <net name="RXD_TTL" class="0">
@@
 <label x="-190.5" y="162.56" size="1.27" layer="95" rot="R180" xref="yes"/>
 </segment>
-</net>
+<segment>
+<pinref part="JP9" gate="G$1" pin="1"/>
+<wire x1="-195.58" y1="180.34" x2="-190.5" y2="180.34" width="0.1524" layer="91"/>
+<label x="-190.5" y="180.34" size="1.27" layer="95" xref="yes"/>
+</segment>
+</net>
